Commit message: Sync updated robot description files

File: assets/h1_2/h1_2_ros.urdf (robot description, URDF)
Before this commit: robot h1_2, 60 links, 59 joints
Links:
- link left_ankle_pitch_link: geometry visual mesh filename=package://h12_ros2_model/assets/h1_2/meshes/left_ankle_pitc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
- link left_hip_pitch_link: geometry collision mesh filename=package://h12_ros2_model/assets/h1_2/meshes/left_hip_pitch_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; visual mesh filename=package://h12_ros2_model/assets/h1_2/meshes/left_hip_pitch_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
- link left_hip_roll_link: geometry collision mesh filename=package://h12_ros2_model/assets/h1_2/meshes/left_hip_roll_l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; visual mesh filename=package://h12_ros2_model/assets/h1_2/meshes/left_hip_roll_l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
- link left_hip_yaw_link: geometry visual mesh filename=package://h12_ros2_model/assets/h1_2/meshes/left_hip_yaw_li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
- link left_knee_link: geometry collision cylinder length=0.2 radius=0.04; visual mesh filename=package://h12_ros2_model/assets/h1_2/meshes/left_knee_link.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
- link pelvis: geometry collision mesh filename=package://h12_ros2_model/assets/h1_2/meshes/pelvis.STL; visual mesh filename=package://h12_ros2_model/assets/h1_2/meshes/pelvis.STL
- link right_ankle_pitch_link: geometry visual mesh filename=package://h12_ros2_model/assets/h1_2/meshes/right_ankle_pit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
- link right_hip_pitch_link: geometry collision mesh filename=package://h12_ros2_model/assets/h1_2/meshes/right_hip_pitch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; visual mesh filename=package://h12_ros2_model/assets/h1_2/meshes/right_hip_pitch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
- link right_hip_roll_link: geometry collision mesh filename=package://h12_ros2_model/assets/h1_2/meshes/right_hip_roll_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; visual mesh filename=package://h12_ros2_model/assets/h1_2/meshes/right_hip_roll_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
- link right_hip_yaw_link: geometry visual mesh filename=package://h12_ros2_model/assets/h1_2/meshes/right_hip_yaw_l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
- link right_knee_link: geometry collision cylinder length=0.2 radius=0.04; visual mesh filename=package://h12_ros2_model/assets/h1_2/meshes/right_knee_link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
- link torso_link: geometry collision mesh filename=package://h12_ros2_model/assets/h1_2/meshes/torso_link.STL; visual mesh filename=package://h12_ros2_model/assets/h1_2/meshes/torso_link.STL
